File: learn_smd.sch (EAGLE design)
At the start: 11 parts, among them Q1 MMBT2222A, Q2 MMBT2222A

Commit message: switched to through hole battery
Parts:
- removed BAT1: (no value), SparkFun-Electromechanical:BATTERY20SMD
- added BT1: BAT-HLD-001-THM, BAT-HLD-001-THM:BAT-HLD-001-THM
Connections:
- net GND: now also BT1.-; no longer BAT1.-
- net N$6: now also BT1.+; no longer BAT1.+
Changed lines of the file:
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@@
 <setting verticaltext="up"/>
 </settings>
-<grid distance="0.1" unitdist="inch" unit="inch" style="lines" multiple="1" display="yes" altdistance="0.01" altunitdist="inch" altunit="inch"/>
+<grid distance="0.1" unitdist="inch" unit="inch" style="lines" multiple="1" display="no" altdistance="0.01" altunitdist="inch" altunit="inch"/>
 <layers>
 <layer number="1" name="Top" color="4" fill="1" visible="no" active="no"/>
@@
 <part name="GND2" library="SparkFun-Aesthetics" deviceset="GND" device=""/>
 <part name="GND3" library="SparkFun-Aesthetics" deviceset="GND" device=""/>
-<part name="BAT1" library="SparkFun-Electromechanical" deviceset="BATTERY" device="20SMD"/>
+<part name="BT1" library="BAT-HLD-001-THM" deviceset="BAT-HLD-001-THM" device="">
+<attribute name="COST1000" value="0.196"/>
+<attribute name="COST1000_B" value="0.184"/>
+<attribute name="LINK" value="http://www.mouser.com/ProductDetail/Linx-Technologies/BAT-HLD-001-THM/"/>
+<attribute name="LINK_B" value="http://www.mouser.com/ProductDetail/Panasonic-Battery/CR2016/"/>
+</part>
 </parts>
 <sheets>
@@
 <instance part="GND2" gate="1" x="106.68" y="35.56"/>
 <instance part="GND3" gate="1" x="38.1" y="63.5"/>
-<instance part="BAT1" gate="G$1" x="38.1" y="76.2" rot="R270"/>
+<instance part="BT1" gate="G$1" x="38.1" y="76.2" smashed="yes" rot="R90">
+<attribute name="COST1000" x="38.1" y="76.2" size="1.778" layer="96" rot="R90" display="off"/>
+<attribute name="LINK" x="38.1" y="76.2" size="1.778" layer="96" rot="R90" display="off"/>
+<attribute name="COST1000_B" x="38.1" y="76.2" size="1.778" layer="96" rot="R90" display="off"/>
+<attribute name="LINK_B" x="38.1" y="76.2" size="1.778" layer="96" rot="R90" display="off"/>
+<attribute name="NAME" x="34.925" y="74.93" size="1.778" layer="95" rot="R90" display="off"/>
+<attribute name="VALUE" x="43.18" y="74.93" size="1.778" layer="96" rot="R90" display="off"/>
+</instance>
 </instances>
 <busses>
@@
 <wire x1="88.9" y1="71.12" x2="88.9" y2="91.44" width="0.1524" layer="91"/>
 <junction x="88.9" y="91.44"/>
-<pinref part="BAT1" gate="G$1" pin="+"/>
 <wire x1="38.1" y1="81.28" x2="38.1" y2="91.44" width="0.1524" layer="91"/>
 <wire x1="38.1" y1="91.44" x2="53.34" y2="91.44" width="0.1524" layer="91"/>
 <junction x="53.34" y="91.44"/>
+<pinref part="BT1" gate="G$1" pin="+"/>
 </segment>
 </net>
@@
 <segment>
 <pinref part="GND3" gate="1" pin="GND"/>
-<pinref part="BAT1" gate="G$1" pin="-"/>
 <wire x1="38.1" y1="66.04" x2="38.1" y2="71.12" width="0.1524" layer="91"/>
-</segment>
-</net>
+<pinref part="BT1" gate="G$1" pin="-"/>
+</segment>
+</net>
